File: Hardware/0. Project/WeatherLog.sch (EAGLE design)
At the start: 84 parts, among them IC2 TP4056, IC4 DW01A-G, Q1 BC817, Q2 26MHz ±10ppm, Q3 BC817, Q4 BC817, U1 ESP8266EX, U10 VEML6070, U2 FS8205A, U3 FT232RL, U4 RT9193-33GB, U5 25Q80ASSIG, U6 BMP280, U7 DS3231/SO, U8 SI7021, U9 TSL2561FN, X3 USB Micro B

Commit message: Schematic sheet renumbered
Parts:
- removed D4: BAT760, diode:DIODE-SOD323-W
- removed IC2: TP4056, TP4056:TP4056
- removed IC4: DW01A-G, DW01A-G:DW01A-G
- removed LED6: RGBLED5050, adafruit:RGBLED5050
- removed R34, R35: 4k7 (5%), rcl:R-EU_R0603
- removed R36: 1k (5%), rcl:R-EU_R0603
- removed R38, R39: 10k (5%), rcl:R-EU_R0603
- removed X3: USB Micro B, Micro USB Connector:ZX62D-B-5PA8
- added D1: BAT760, diode:DIODE-SOD323-W
- added LED1: (no value), led:LED3MM
- added R22: 20R, rcl:R-EU_R0603
- added R23: 10k, rcl:R-EU_R0603
- added R24, R26: 4k7 (5%), rcl:R-EU_R0603
- added R25: 499R (1%), rcl:R-EU_R0603
- added U11: TSL2561FN, TSL2561:TSL2561FN
- added U12: VEML6070, VEML6070:VEML6070
- added X1: USB Micro B, Micro USB Connector:ZX62D-B-5PA8
- C10, C11: value 6.8pF -> 100nF
- C13: value 100nF -> 10UF
- C14: value 2.4pF -> 1uF; device rcl:C-EUC0603 -> rcl:C-EUC0805
- C16: value 100nF -> 2.4pF
- C17: value 1uF -> 22nF; device rcl:C-EUC0603 -> rcl:C-EUC0805
- C18: value 10uF -> 1000uF x 10V; device rcl:C-EUC0603 -> rcl:CPOL-EUE2-5
- C19: value 1000uF x 10V -> 100nF; device rcl:CPOL-EUE2-5 -> rcl:C-EUC0805
- C2: value 1uF -> 100nF; device rcl:C-EUC0805 -> rcl:C-EUC0603
- C5: value 10UF -> 10uF
- C6: value 100nF -> 1uF
- C8: value 100nF -> 6.8pF; device rcl:C-EUC0805 -> rcl:C-EUC0603
- C9: value 22nF -> 6.8pF; device rcl:C-EUC0805 -> rcl:C-EUC0603
- LED3: value (none) -> RGBLED5050; device led:LED3MM -> adafruit:RGBLED5050
- Q2: value 26MHz ±10ppm -> BC817; device Crystal (SMD):KX-7 -> transistor-npn:BC817-40LT1SMD
- Q3: value BC817 -> 26MHz ±10ppm; device transistor-npn:BC817-40LT1SMD -> Crystal (SMD):KX-7
- R1: value 10k -> 270R; device rcl:R-EU_R0603 -> rcl:R-EU_0204/7
- R10: value 10k -> 100R; device ptc-ntc:NTC640 -> rcl:R-EU_R0603
- R11: value 5k -> 12k (1%); device resistor:R-TRIMM64P -> rcl:R-EU_R0603
- R12: value 12k (1%) -> 10k (5%)
- R14: value 499R (1%) -> 200R
- R15: device rcl:R-EU_R0603 -> rcl:R-EU_M0805
- R16: value 10k (5%) -> 330k (5%)
- R17: value 10k (5%) -> 100k (5%); device rcl:R-EU_M0805 -> rcl:R-EU_R0603
- R18: value 330k (5%) -> 100k
- R19: value 100k (5%) -> 10k (5%)
- R2: value 20R -> 270R; device rcl:R-EU_R0603 -> rcl:R-EU_0204/7
- R20, R21: value 270R -> 1k; device rcl:R-EU_0204/7 -> rcl:R-EU_R0603
- R3: value 1k -> 1k2 (5%)
- R4: value 100R -> 1k (5%)
- R5: value 1k2 (5%) -> 5k; device rcl:R-EU_R0603 -> resistor:R-TRIMM64P
- R6: value 100k -> 10k (5%)
- R7: value 200R -> 10k; device rcl:R-EU_R0603 -> ptc-ntc:NTC640
- R8: value 1k -> 10k (5%)
- U1: value ESP8266EX -> TP4056; device ESP8266EX:ESP8266EX -> TP4056:TP4056
- U10: value VEML6070 -> SI7021; device VEML6070:VEML6070 -> SI7021:SI7021
- U2: value FS8205A -> FT232RL; device FS8205A:FS8205A -> FT232RL:FT232RL
- U3: value FT232RL -> DW01A-G; device FT232RL:FT232RL -> DW01A-G:DW01A-G
- U4: value RT9193-33GB -> FS8205A; device RT9193-33GB:RT9193-33GB -> FS8205A:FS8205A
- U5: value 25Q80ASSIG -> ESP8266EX; device 25Q80ASSIG:25Q80ASSIG -> ESP8266EX:ESP8266EX
- U6: value BMP280 -> 25Q80ASSIG; device BMP280:BMP280 -> 25Q80ASSIG:25Q80ASSIG
- U7: value DS3231/SO -> RT9193-33GB; device adafruit:DS3231/SO -> RT9193-33GB:RT9193-33GB
- U8: value SI7021 -> DS3231/SO; device SI7021:SI7021 -> adafruit:DS3231/SO
- U9: value TSL2561FN -> BMP280; device TSL2561:TSL2561FN -> BMP280:BMP280
Connections:
- net !BAT_CHARGING!: now also LED3.GREEN_C, U1.!CHRG; no longer IC2.!CHRG, LED6.GREEN_C
- net !BAT_STANDBY!: now also LED3.BLUE_C, U1.!STDBY; no longer IC2.!STDBY, LED6.BLUE_C
- net !ESP_PROG_MODE!: now also Q2.C, R27.1, U5.GPIO0; no longer Q4.C, R16.1, U1.GPIO0
- net !ESP_RESET!: now also C10.2, Q1.C, R12.1, U5.!EXT_RSTB; no longer C12.2, Q3.C, R13.1, U1.!EXT_RSTB
- net 3.3V: now also C12.2, C18.+, C19.2, C4.2, C5.2, C6.2, R12.2, R19.2, R24.2, R26.2, U11.VDD, U12.VDD, U5.VDD3P3, U5.VDDA, U5.VDDD, U5.VDDPST, U6.VCC, U7.VOUT, U9.VDDIO; no longer C13.2, C16.2, C17.2, C18.2, C19.+, C8.2, R15.2, R16.2, R34.2, R35.2, U1.VDD3P3, U1.VDDA, U1.VDDD, U1.VDDPST, U4.VOUT, U5.VCC, U6.VDD, U6.VDDIO, U7.VDD
- net BAT_OVER_CHARGE_DETECTED: now also U3.OC, U4.G2; no longer IC4.OC, U2.G2
- net BAT_OVER_DISCHARGE_DETECTED: now also R23.2, U3.OD, U4.G1; no longer IC4.OD, R1.2, U2.G1
- net DTR: now also Q2.E, R6.2, U2.!DTR!; no longer Q4.E, R38.2, U3.!DTR!
- net ESP_ENABLE: now also C11.2, R13.1, U5.CHIP_EN; no longer C1.2, R15.1, U1.CHIP_EN
- net ESP_I2C_SCL: now also R26.1, U11.SCL, U12.SCL, U5.GPIO5, U9.SCL/SCLK; no longer R35.1, U1.GPIO5, U6.SCL/SCLK, U7.SCL, U9.SCL
- net ESP_I2C_SDA: now also R24.1, U11.SDA, U12.SDA, U5.(PWM3)GPIO4, U9.SDA/MISO; no longer R34.1, U1.(PWM3)GPIO4, U6.SDA/MISO, U7.SDA, U9.SDA
- net ESP_ICSP_UART_RX: now also U2.TXD, U5.U0RXD; no longer U1.U0RXD, U3.TXD
- net ESP_ICSP_UART_TX: now also R25.2, U2.RXD; no longer R14.2, U3.RXD
- net GND: now also C13.2, C14.2, C17.2, C18.-, C19.1, C3.1, C4.1, C5.1, C9.1, Q3.GND, R11.1, R15.2, R17.1, R18.1, R5.A, R5.S, R7.1, R9.1, U11.ADDR, U11.GND, U12.GND, U2.AGND, U2.GND1, U2.GND2, U2.GND3, U2.TEST, U4.S2_1, X1G$1.4, X1G$1.5; no longer C13.1, C14.1, C17.1, C18.1, C19.-, C4.2, C5.2, C7.1, C9.2, IC2.GND, Q2.GND, R10.1, R11.A, R11.S, R12.1, R17.2, R19.1, R5.1, R6.1, U2.S2_1, U3.AGND, U3.GND1, U3.GND2, U3.GND3, U3.TEST, U4.GND, U9.ADDR, X3G$1.4, X3G$1.5
- net N$1: now also Q4.B, R23.1; no longer Q1.B, R1.1
- net N$10: now also LED3.GREEN_A, R21.1; no longer LED6.GREEN_A, R8.1
- net N$11: now also C8.2, Q3.1, U5.XTAL_OUT; no longer C11.2, Q2.1, U1.XTAL_OUT
- net N$12: now also LED3.BLUE_A, R20.1; no longer LED6.BLUE_A, R9.1
- net N$13: now also R14.1, U6.!CS!; no longer R7.1, U5.!CS!
- net N$14: now also U5.SPI_CLK, U6.SCLK; no longer U1.SPI_CLK, U5.SCLK
- net N$15: now also U5.SPI_HD, U6.!HOLD!; no longer U1.SPI_HD, U5.!HOLD!
- net N$16: now also R4.1, R5.E, R7.2, U1.TEMP1; no longer IC2.TEMP1, R10.2, R11.E, R36.1
- net N$17: now also R2.1, U2.CBUS0; no longer R20.1, U3.CBUS0
- net N$18: now also R16.1, R17.2, U5.TOUT; no longer R18.1, R19.2, U1.TOUT
- net N$19: now also R1.1, U2.CBUS1; no longer R21.1, U3.CBUS1
- net N$2: now also R14.2, U5.SPI_CS0; no longer R7.2, U1.SPI_CS0
- net N$20: now also Q2.B, R8.2; no longer Q4.B, R39.2
- net N$21: now also U5.SPI_MOSI, U6.MISO; no longer U1.SPI_MOSI, U5.MISO
- net N$23: now also U5.SPI_MISO, U6.MOSI; no longer U1.SPI_MISO, U5.MOSI
- net N$24: now also U5.LNA; no longer U1.LNA
- net N$25: now also R11.2, U5.RES12K; no longer R12.2, U1.RES12K
- net N$26: now also U5.SPI_WP, U6.!WP!; no longer U1.SPI_WP, U5.!WP!
- net N$27: now also C9.2, Q3.2, U5.XTAL_IN; no longer C10.2, Q2.2, U1.XTAL_IN
- net N$28: now also R25.1, U5.U0TXD; no longer R14.1, U1.U0TXD
- net N$29: now also C16.2; no longer C14.2
- net N$3: now also LED3.RED_C, Q4.C; no longer LED6.RED_C, Q1.C
- net N$30: now also R28.1, U8.!INT!/SQW; no longer R27.1, U7.!INT!/SQW
- net N$31: now also R15.1, U5.(GPIO15/SPI_CS/U0RTS/PWM1)MTDO; no longer R17.1, U1.(GPIO15/SPI_CS/U0RTS/PWM1)MTDO
- net N$32: now also R33.1, U8.32KHZ; no longer R28.1, U7.32KHZ
- net N$33: now also U11.INT; no longer U9.INT
- net N$34: now also R31.1, U9.MOSI; no longer R30.1, U6.MOSI
- net N$35: now also R30.1, U12.ACK; no longer R31.1, U10.ACK
- net N$36: now also U12.RST; no longer U10.RST
- net N$37: now also R19.1, U5.(U1TXD)GPIO2; no longer R33.1, U1.(U1TXD)GPIO2
- net N$4: now also C17.1, U7.BP; no longer C9.1, U4.BP
- net N$49: now also R2.2; no longer R20.2
- net N$5: now also LED3.RED_A, R22.1; no longer LED6.RED_A, R2.1
- net N$50: now also LED1.C, R1.2; no longer LED3.C, R21.2
- net N$53: now also U2.USBDM, X1G$1.2; no longer U3.USBDM, X3G$1.2
- net N$54: now also U2.USBDP, X1G$1.3; no longer U3.USBDP, X3G$1.3
- net N$59: now also Q1.B, R6.1; no longer Q3.B, R38.1
- net N$6: now also R3.2, U1.PROG2; no longer IC2.PROG2, R5.2
- net N$7: now also R9.2, U3.CS; no longer IC4.CS, R3.2
- net N$8: now also C7.1, R10.2, U3.VCC; no longer C3.1, IC4.VCC, R4.2
- net N$9: now also U8.VBAT; no longer U7.VBAT
- net RTS: now also Q1.E, R8.1, U2.!RTS!; no longer Q3.E, R39.1, U3.!RTS!
- net VCC_IO: now also C3.2, LED1.A, U2.3V3OUT, U2.VCCIO; no longer C6.2, LED3.A, U3.3V3OUT, U3.VCCIO
- net VUSB1: now also C1.2, D1.A, X1G$1.1; no longer C7.2, D4.A, X3G$1.1
- net V_BAT+: now also C13.1, C14.1, R10.1, R16.2, R22.2, U1.BAT, U7.EN, U7.VIN; no longer C2.1, C5.1, IC2.BAT, R2.2, R4.1, R6.2, U4.EN, U4.VIN
- net V_BAT-: now also C7.2, Q4.E, U3.GND, U4.S1_1; no longer C3.2, IC4.GND, Q1.E, U2.S1_1
- net V_EXTERNAL_SUPPLY: now also C2.1, D1.C, R20.2, R21.2, R4.2, U1.CE, U1.VCC, U2.VCC; no longer C4.1, D4.C, IC2.CE, IC2.VCC, R36.2, R8.2, R9.2, U3.VCC
Other:
- moved on the sheet: A1, C1, C10, C11, C12, C13, C14, C15, C16, C17, C2, C20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
